Commit message: added cameras to robot

File: robot_description/base.urdf.xacro (robot description, xacro)
@@ -17,5 +17,9 @@
   <xacro:include filename="$(find store_gfk)/robot_description/custom/support.urdf.xacro"/>
   <!-- RGBD cameras -->
-<!--  <xacro:include filename="$(find store_gfk)/robot_description/custom/RGBDs.urdf.xacro"/>-->
+    <xacro:include filename="$(find store_gfk)/robot_description/custom/cameras/cameras.urdf.xacro"/>
+  <!-- RGB -->
+  <!--  <xacro:include filename="$(find store_gfk)/robot_description/custom/elp_rgb.urdf.xacro"/>-->
+  <!-- -D -->
+  <!--  <xacro:include filename="$(find store_gfk)/robot_description/custom/structure_sensor.urdf.xacro"/>-->
   <!-- Wheel characteristics -->
   <xacro:property name="wheel_radius"     value="0.0985"/>
@@ -86,6 +90,8 @@
       <origin xyz="-0.201 -0.1062 0.195" rpy="0 0 0"/>
     </xacro:antenna>
-<!-- support -->
-<xacro:support name="${name}_support" parent="${name}_link"/>
+    <!-- support -->
+    <xacro:support name="${name}_support" parent="${name}_link"/>
+    <!-- cameras -->
+<!--    <xacro:support name="${name}_camera" parent="${name}_support"/>-->
     <!-- IMU -->
     <!-- @todo pmb2_hardware_gazebo needs an IMU!  -->

File: robot_description/custom/support.urdf.xacro (robot description, xacro)
@@ -22,4 +22,10 @@
 		  </geometry>
 		</visual>
+      <collision>
+  		  <origin xyz="0 0 ${c/2}" rpy="0 0 0"/>
+		  <geometry>
+		    <box size="0.3 0.15 ${c}"/>
+		  </geometry>
+      </collision>
 	  </link>
     <joint name="support_joint" type="fixed">
