Commit message: refactored a bit, issue on vel overload

File: robot_description/custom/cameras/cameras.urdf.xacro (robot description, xacro)
@@ -17,5 +17,5 @@
   <xacro:property name="tl_rgbd_y" value="${support_y/2}"/>
   <xacro:property name="tl_rgbd_z" value="${2/3*support_height+robot_height}"/>
-  <xacro:property name="tl_rgbd_R" value="0.0"/> <!-- rotations are with respect ?? axis-->
+  <xacro:property name="tl_rgbd_R" value="20.0"/> <!-- rotations are with respect world axis-->
   <xacro:property name="tl_rgbd_P" value="0.0"/>
   <xacro:property name="tl_rgbd_Y" value="90.0"/>
@@ -24,5 +24,5 @@
   <xacro:property name="tr_rgbd_y" value="${-support_y/2}"/>
   <xacro:property name="tr_rgbd_z" value="${2/3*support_height+robot_height}"/>
-  <xacro:property name="tr_rgbd_R" value="0.0"/> <!-- rotations are with respect ?? axis-->
+  <xacro:property name="tr_rgbd_R" value="-20.0"/>
   <xacro:property name="tr_rgbd_P" value="0.0"/>
   <xacro:property name="tr_rgbd_Y" value="-90.0"/>
@@ -32,5 +32,5 @@
   <xacro:property name="bl_rgbd_y" value="${support_y/2}"/>
   <xacro:property name="bl_rgbd_z" value="${1/3*support_height+robot_height}"/>
-  <xacro:property name="bl_rgbd_R" value="0.0"/> <!-- rotations are with respect ?? axis-->
+  <xacro:property name="bl_rgbd_R" value="-20.0"/>
   <xacro:property name="bl_rgbd_P" value="0.0"/>
   <xacro:property name="bl_rgbd_Y" value="90.0"/>
@@ -39,5 +39,5 @@
   <xacro:property name="br_rgbd_y" value="${-support_y/2}"/>
   <xacro:property name="br_rgbd_z" value="${1/3*support_height+robot_height}"/>
-  <xacro:property name="br_rgbd_R" value="0.0"/> <!-- rotations are with respect ?? axis-->
+  <xacro:property name="br_rgbd_R" value="20.0"/>
   <xacro:property name="br_rgbd_P" value="0.0"/>
   <xacro:property name="br_rgbd_Y" value="-90.0"/>

Commit message: fixed camera orientation, working alignment

File: robot_description/custom/cameras/cameras.urdf.xacro (robot description, xacro)
@@ -17,6 +17,6 @@
   <xacro:property name="tl_rgbd_y" value="${support_y/2}"/>
   <xacro:property name="tl_rgbd_z" value="${2/3*support_height+robot_height}"/>
-  <xacro:property name="tl_rgbd_R" value="20.0"/> <!-- rotations are with respect world axis-->
-  <xacro:property name="tl_rgbd_P" value="0.0"/>
+  <xacro:property name="tl_rgbd_R" value="0.0"/> <!-- rotations are with respect world axis-->
+  <xacro:property name="tl_rgbd_P" value="-15.0"/>
   <xacro:property name="tl_rgbd_Y" value="90.0"/>
   <!-- top-right camera -->
@@ -24,6 +24,6 @@
   <xacro:property name="tr_rgbd_y" value="${-support_y/2}"/>
   <xacro:property name="tr_rgbd_z" value="${2/3*support_height+robot_height}"/>
-  <xacro:property name="tr_rgbd_R" value="-20.0"/>
-  <xacro:property name="tr_rgbd_P" value="0.0"/>
+  <xacro:property name="tr_rgbd_R" value="0.0"/>
+  <xacro:property name="tr_rgbd_P" value="15.0"/>
   <xacro:property name="tr_rgbd_Y" value="-90.0"/>
   <!-- next not used if two cameras only -->
@@ -32,6 +32,6 @@
   <xacro:property name="bl_rgbd_y" value="${support_y/2}"/>
   <xacro:property name="bl_rgbd_z" value="${1/3*support_height+robot_height}"/>
-  <xacro:property name="bl_rgbd_R" value="-20.0"/>
-  <xacro:property name="bl_rgbd_P" value="0.0"/>
+  <xacro:property name="bl_rgbd_R" value="0.0"/>
+  <xacro:property name="bl_rgbd_P" value="-15.0"/>
   <xacro:property name="bl_rgbd_Y" value="90.0"/>
   <!-- bottom-right camera -->
@@ -39,6 +39,6 @@
   <xacro:property name="br_rgbd_y" value="${-support_y/2}"/>
   <xacro:property name="br_rgbd_z" value="${1/3*support_height+robot_height}"/>
-  <xacro:property name="br_rgbd_R" value="20.0"/>
-  <xacro:property name="br_rgbd_P" value="0.0"/>
+  <xacro:property name="br_rgbd_R" value="0.0"/>
+  <xacro:property name="br_rgbd_P" value="15.0"/>
   <xacro:property name="br_rgbd_Y" value="-90.0"/>
   <!-- base RGBD characteristics -->

Commit message: working rotation and capture

File: robot_description/custom/cameras/cameras.urdf.xacro (robot description, xacro)
@@ -18,5 +18,5 @@
   <xacro:property name="tl_rgbd_z" value="${2/3*support_height+robot_height}"/>
   <xacro:property name="tl_rgbd_R" value="0.0"/> <!-- rotations are with respect world axis-->
-  <xacro:property name="tl_rgbd_P" value="-15.0"/>
+  <xacro:property name="tl_rgbd_P" value="-10.0"/><!-- -10.0-->
   <xacro:property name="tl_rgbd_Y" value="90.0"/>
   <!-- top-right camera -->
@@ -25,5 +25,5 @@
   <xacro:property name="tr_rgbd_z" value="${2/3*support_height+robot_height}"/>
   <xacro:property name="tr_rgbd_R" value="0.0"/>
-  <xacro:property name="tr_rgbd_P" value="15.0"/>
+  <xacro:property name="tr_rgbd_P" value="-10.0"/><!-- -10.0-->
   <xacro:property name="tr_rgbd_Y" value="-90.0"/>
   <!-- next not used if two cameras only -->
@@ -33,5 +33,5 @@
   <xacro:property name="bl_rgbd_z" value="${1/3*support_height+robot_height}"/>
   <xacro:property name="bl_rgbd_R" value="0.0"/>
-  <xacro:property name="bl_rgbd_P" value="-15.0"/>
+  <xacro:property name="bl_rgbd_P" value="10.0"/><!-- 10.0-->
   <xacro:property name="bl_rgbd_Y" value="90.0"/>
   <!-- bottom-right camera -->
@@ -40,5 +40,5 @@
   <xacro:property name="br_rgbd_z" value="${1/3*support_height+robot_height}"/>
   <xacro:property name="br_rgbd_R" value="0.0"/>
-  <xacro:property name="br_rgbd_P" value="15.0"/>
+  <xacro:property name="br_rgbd_P" value="10.0"/><!-- 10.0-->
   <xacro:property name="br_rgbd_Y" value="-90.0"/>
   <!-- base RGBD characteristics -->

File: robot_description/custom/cameras/rgbd_camera.gazebo.xacro (robot description, xacro)
@@ -53,9 +53,9 @@
         <update_rate>6.0</update_rate>
         <camera>
-          <horizontal_fov>${58.0 * deg_to_rad}</horizontal_fov>
+          <horizontal_fov>${60.0 * deg_to_rad}</horizontal_fov> <!-- 58.0 -->
           <image>
             <format>R8G8B8</format>
-            <width>320</width>
-            <height>240</height>
+            <width>3840</width> <!-- 320 -->
+            <height>2880</height> <!-- 240 , 2160 stockbot, 2880 to have 4/3 aspect ratio-->
           </image>
           <clip>

Commit message: finished repulsing, giving goals

File: robot_description/custom/cameras/cameras.urdf.xacro (robot description, xacro)
@@ -18,5 +18,5 @@
   <xacro:property name="tl_rgbd_z" value="${2/3*support_height+robot_height}"/>
   <xacro:property name="tl_rgbd_R" value="0.0"/> <!-- rotations are with respect world axis-->
-  <xacro:property name="tl_rgbd_P" value="-10.0"/><!-- -10.0-->
+  <xacro:property name="tl_rgbd_P" value="0.0"/><!-- -10.0-->
   <xacro:property name="tl_rgbd_Y" value="90.0"/>
   <!-- top-right camera -->
@@ -25,5 +25,5 @@
   <xacro:property name="tr_rgbd_z" value="${2/3*support_height+robot_height}"/>
   <xacro:property name="tr_rgbd_R" value="0.0"/>
-  <xacro:property name="tr_rgbd_P" value="-10.0"/><!-- -10.0-->
+  <xacro:property name="tr_rgbd_P" value="0.0"/><!-- -10.0-->
   <xacro:property name="tr_rgbd_Y" value="-90.0"/>
   <!-- next not used if two cameras only -->
@@ -33,5 +33,5 @@
   <xacro:property name="bl_rgbd_z" value="${1/3*support_height+robot_height}"/>
   <xacro:property name="bl_rgbd_R" value="0.0"/>
-  <xacro:property name="bl_rgbd_P" value="10.0"/><!-- 10.0-->
+  <xacro:property name="bl_rgbd_P" value="0.0"/><!-- 10.0-->
   <xacro:property name="bl_rgbd_Y" value="90.0"/>
   <!-- bottom-right camera -->
@@ -40,5 +40,5 @@
   <xacro:property name="br_rgbd_z" value="${1/3*support_height+robot_height}"/>
   <xacro:property name="br_rgbd_R" value="0.0"/>
-  <xacro:property name="br_rgbd_P" value="10.0"/><!-- 10.0-->
+  <xacro:property name="br_rgbd_P" value="0.0"/><!-- 10.0-->
   <xacro:property name="br_rgbd_Y" value="-90.0"/>
   <!-- base RGBD characteristics -->

Commit message: fixed wrong height calculation

File: robot_description/custom/cameras/cameras.urdf.xacro (robot description, xacro)
@@ -5,9 +5,9 @@
 <!--<xacro:include filename="$(find store_gfk)/robot_description/custom/cameras/elp_rgb.urdf.xacro"/>-->
   <!-- TODO: inherit them from support file -->
-  <xacro:property name="robot_height"   value="0.195"/>
-  <xacro:property name="support_height"   value="1.6"/>
+  <xacro:property name="base_height"   value="0.195"/>
+  <xacro:property name="robot_height"   value="1.8"/>
   <xacro:property name="support_x"   value="0.3"/> <!-- support length on x-->
   <xacro:property name="support_y"   value="0.15"/> <!-- support length on y-->
-  <xacro:property name="support_z"   value="${support_height-robot_height}"/> <!-- support length on z-->
+  <xacro:property name="support_z"   value="${robot_height-base_height}"/> <!-- support height-->
   <!-- cameras config -->
   <xacro:property name="n_cameras" value="four"/>
@@ -16,5 +16,5 @@
   <xacro:property name="tl_rgbd_x" value="0.0"/>
   <xacro:property name="tl_rgbd_y" value="${support_y/2}"/>
-  <xacro:property name="tl_rgbd_z" value="${2/3*support_height+robot_height}"/>
+  <xacro:property name="tl_rgbd_z" value="${2/3*robot_height + base_height}"/>
   <xacro:property name="tl_rgbd_R" value="0.0"/> <!-- rotations are with respect world axis-->
   <xacro:property name="tl_rgbd_P" value="0.0"/><!-- -10.0-->
@@ -23,5 +23,5 @@
   <xacro:property name="tr_rgbd_x" value="0.0"/>
   <xacro:property name="tr_rgbd_y" value="${-support_y/2}"/>
-  <xacro:property name="tr_rgbd_z" value="${2/3*support_height+robot_height}"/>
+  <xacro:property name="tr_rgbd_z" value="${2/3*robot_height + base_height}"/>
   <xacro:property name="tr_rgbd_R" value="0.0"/>
   <xacro:property name="tr_rgbd_P" value="0.0"/><!-- -10.0-->
@@ -31,5 +31,5 @@
   <xacro:property name="bl_rgbd_x" value="0.0"/>
   <xacro:property name="bl_rgbd_y" value="${support_y/2}"/>
-  <xacro:property name="bl_rgbd_z" value="${1/3*support_height+robot_height}"/>
+  <xacro:property name="bl_rgbd_z" value="${1/3*robot_height}"/>
   <xacro:property name="bl_rgbd_R" value="0.0"/>
   <xacro:property name="bl_rgbd_P" value="0.0"/><!-- 10.0-->
@@ -38,5 +38,5 @@
   <xacro:property name="br_rgbd_x" value="0.0"/>
   <xacro:property name="br_rgbd_y" value="${-support_y/2}"/>
-  <xacro:property name="br_rgbd_z" value="${1/3*support_height+robot_height}"/>
+  <xacro:property name="br_rgbd_z" value="${1/3*robot_height}"/>
   <xacro:property name="br_rgbd_R" value="0.0"/>
   <xacro:property name="br_rgbd_P" value="0.0"/><!-- 10.0-->

File: robot_description/custom/support.urdf.xacro (robot description, xacro)
@@ -1,29 +1,30 @@
 <?xml version="1.0"?>
 <robot xmlns:xacro="http://ros.org/wiki/xacro">
-  <xacro:property name="robot_height"   value="0.195"/>
-  <xacro:property name="support_height"   value="1.6"/>
+ <!-- the fixed joint for the support is at the top of the base-->
+  <xacro:property name="base_height"   value="0.195"/>
+  <xacro:property name="robot_height"   value="1.8"/>
   <xacro:property name="support_mass"   value="2"/>
-  <xacro:property name="a"   value="0.3"/> <!-- support length on x-->
-  <xacro:property name="b"   value="0.15"/> <!-- support length on y-->
-  <xacro:property name="c"   value="${support_height-robot_height}"/> <!-- support length on z-->
+  <xacro:property name="support_x"   value="0.3"/> <!-- support length on x-->
+  <xacro:property name="support_y"   value="0.15"/> <!-- support length on y-->
+  <xacro:property name="support_z"   value="${robot_height-base_height}"/> <!-- support height-->
   <xacro:macro name="support" params="name parent">
 	<link name="${name}_link">
        <inertial>
-        <origin xyz="0 0 ${c/2}" rpy="0 0 0"/>
+        <origin xyz="0 0 ${support_z/2}" rpy="0 0 0"/>
         <mass value="${support_mass}"/>
-        <inertia ixx="${1/12*support_mass*(b*b+c*c)}" ixy="0.0" ixz="0.0"
-                 iyy="${1/12*support_mass*(a*a+c*c)}" iyz="0.0"
-                 izz="${1/12*support_mass*(a*a+b*b)}"/>
+        <inertia ixx="${1/12*support_mass*(support_y*support_y+support_z*support_z)}" ixy="0.0" ixz="0.0"
+                 iyy="${1/12*support_mass*(support_x*support_x+support_z*support_z)}" iyz="0.0"
+                 izz="${1/12*support_mass*(support_x*support_x+support_y*support_y)}"/>
       </inertial>
 		<visual>
-		  <origin xyz="0 0 ${c/2}" rpy="0 0 0"/>
+		  <origin xyz="0 0 ${support_z/2}" rpy="0 0 0"/>
 		  <geometry>
-		    <box size="0.3 0.15 ${c}"/>
+		    <box size="${support_x} ${support_y} ${support_z}"/>
 		  </geometry>
 		</visual>
       <collision>
-  		  <origin xyz="0 0 ${c/2}" rpy="0 0 0"/>
+  		  <origin xyz="0 0 ${support_z/2}" rpy="0 0 0"/>
 		  <geometry>
-		    <box size="0.3 0.15 ${c}"/>
+		    <box size="${support_x} ${support_y} ${support_z}"/>
 		  </geometry>
       </collision>
@@ -32,5 +33,5 @@
       <parent link="${parent}"/>
       <child link="${name}_link"/>
-      <origin xyz="0 0 ${robot_height}" rpy="0 0 0"/>
+      <origin xyz="0 0 ${base_height}" rpy="0 0 0"/>
     </joint>
     <gazebo reference="${name}_link">

Commit message: 3 cameras on each side now

File: robot_description/custom/cameras/cameras.urdf.xacro (robot description, xacro)
@@ -10,11 +10,9 @@
   <xacro:property name="support_y"   value="0.15"/> <!-- support length on y-->
   <xacro:property name="support_z"   value="${robot_height-base_height}"/> <!-- support height-->
-  <!-- cameras config -->
-  <xacro:property name="n_cameras" value="four"/>
 <!--  <xacro:property name="camera_type" value="kinect"/> TODO.-->
   <!-- top-left camera -->
   <xacro:property name="tl_rgbd_x" value="0.0"/>
   <xacro:property name="tl_rgbd_y" value="${support_y/2}"/>
-  <xacro:property name="tl_rgbd_z" value="${2/3*robot_height + base_height}"/>
+  <xacro:property name="tl_rgbd_z" value="${robot_height - base_height}"/>
   <xacro:property name="tl_rgbd_R" value="0.0"/> <!-- rotations are with respect world axis-->
   <xacro:property name="tl_rgbd_P" value="0.0"/><!-- -10.0-->
@@ -23,13 +21,26 @@
   <xacro:property name="tr_rgbd_x" value="0.0"/>
   <xacro:property name="tr_rgbd_y" value="${-support_y/2}"/>
-  <xacro:property name="tr_rgbd_z" value="${2/3*robot_height + base_height}"/>
+  <xacro:property name="tr_rgbd_z" value="${robot_height - base_height}"/>
   <xacro:property name="tr_rgbd_R" value="0.0"/>
   <xacro:property name="tr_rgbd_P" value="0.0"/><!-- -10.0-->
   <xacro:property name="tr_rgbd_Y" value="-90.0"/>
-  <!-- next not used if two cameras only -->
+  <!-- middle-left camera -->
+  <xacro:property name="ml_rgbd_x" value="0.0"/>
+  <xacro:property name="ml_rgbd_y" value="${support_y/2}"/>
+  <xacro:property name="ml_rgbd_z" value="${2/3*robot_height - base_height}"/>
+  <xacro:property name="ml_rgbd_R" value="0.0"/> <!-- rotations are with respect world axis-->
+  <xacro:property name="ml_rgbd_P" value="0.0"/><!-- -10.0-->
+  <xacro:property name="ml_rgbd_Y" value="90.0"/>
+  <!-- middle-right camera -->
+  <xacro:property name="mr_rgbd_x" value="0.0"/>
+  <xacro:property name="mr_rgbd_y" value="${-support_y/2}"/>
+  <xacro:property name="mr_rgbd_z" value="${2/3*robot_height - base_height}"/>
+  <xacro:property name="mr_rgbd_R" value="0.0"/>
+  <xacro:property name="mr_rgbd_P" value="0.0"/><!-- -10.0-->
+  <xacro:property name="mr_rgbd_Y" value="-90.0"/>
   <!-- bottom-left camera -->
   <xacro:property name="bl_rgbd_x" value="0.0"/>
   <xacro:property name="bl_rgbd_y" value="${support_y/2}"/>
-  <xacro:property name="bl_rgbd_z" value="${1/3*robot_height}"/>
+  <xacro:property name="bl_rgbd_z" value="${1/3*robot_height - base_height}"/>
   <xacro:property name="bl_rgbd_R" value="0.0"/>
   <xacro:property name="bl_rgbd_P" value="0.0"/><!-- 10.0-->
@@ -38,5 +49,5 @@
   <xacro:property name="br_rgbd_x" value="0.0"/>
   <xacro:property name="br_rgbd_y" value="${-support_y/2}"/>
-  <xacro:property name="br_rgbd_z" value="${1/3*robot_height}"/>
+  <xacro:property name="br_rgbd_z" value="${1/3*robot_height - base_height}"/>
   <xacro:property name="br_rgbd_R" value="0.0"/>
   <xacro:property name="br_rgbd_P" value="0.0"/><!-- 10.0-->
@@ -63,31 +74,4 @@
   <xacro:property name="rgb_P" value="15.0"/>
   <xacro:property name="rgb_Y" value="0.0   "/>
-<xacro:if value="${n_cameras == 'two'}">
-  <!-- RGBD base -->
-  <xacro:rgbd_camera name="base_rgbd_camera" parent="base">
-    <!-- Pose of sensor frame wrt to base -->
-    <origin
-      xyz="${base_rgbd_x} ${base_rgbd_y} ${base_rgbd_z}"
-	  rpy="0 0 0" />
-<!--      rpy="${base_rgbd_R * deg_to_rad} ${base_rgbd_P * deg_to_rad} ${base_rgbd_Y * deg_to_rad}"/> -->
-    <!-- Pose of optical frame wrt to sensor -->
-    <origin
-      xyz="0 0 0"
-      rpy="${-90 * deg_to_rad} 0 ${-90 * deg_to_rad}"/>
-  </xacro:rgbd_camera>
-  <!-- RGBD roof -->
-  <xacro:rgbd_camera name="roof_rgbd_camera" parent="base">
-    <!-- Pose of sensor frame wrt to base -->
-    <origin
-      xyz="${roof_rgbd_x} ${roof_rgbd_y} ${roof_rgbd_z}"
-      rpy="0 0 0" />
-<!--      rpy="${roof_rgbd_R * deg_to_rad} ${roof_rgbd_P * deg_to_rad} ${roof_rgbd_Y * deg_to_rad}"/>-->
-    <!-- Pose of optical frame wrt to sensor -->
-    <origin
-      xyz="0 0 0"
-      rpy="${-90 * deg_to_rad} 0 ${-90 * deg_to_rad}"/>
-  </xacro:rgbd_camera>
-</xacro:if>
-<xacro:if value="${n_cameras == 'four'}">
   <!-- top-left RGBD -->
   <xacro:rgbd_camera name="tl_rgbd_camera" parent="base">
@@ -107,4 +91,26 @@
       xyz="${tr_rgbd_x} ${tr_rgbd_y} ${tr_rgbd_z}"
   	  rpy="${tr_rgbd_R * deg_to_rad} ${tr_rgbd_P * deg_to_rad} ${tr_rgbd_Y * deg_to_rad}" />
+    <!-- Pose of optical frame wrt to sensor -->
+    <origin
+      xyz="0 0 0"
+      rpy="${-90 * deg_to_rad} 0 ${-90 * deg_to_rad}"/>
+  </xacro:rgbd_camera>
+<!-- middle-left RGBD -->
+  <xacro:rgbd_camera name="ml_rgbd_camera" parent="base">
+    <!-- Pose of sensor frame wrt to base -->
+    <origin
+      xyz="${ml_rgbd_x} ${ml_rgbd_y} ${ml_rgbd_z}"
+	  rpy="${ml_rgbd_R * deg_to_rad} ${ml_rgbd_P * deg_to_rad} ${ml_rgbd_Y * deg_to_rad}" />
+    <!-- Pose of optical frame wrt to sensor -->
+    <origin
+      xyz="0 0 0"
+      rpy="${-90 * deg_to_rad} 0 ${-90 * deg_to_rad}"/>
+  </xacro:rgbd_camera>
+  <!-- middle-right RGBD -->
+  <xacro:rgbd_camera name="mr_rgbd_camera" parent="base">
+    <!-- Pose of sensor frame wrt to base -->
+    <origin
+      xyz="${mr_rgbd_x} ${mr_rgbd_y} ${mr_rgbd_z}"
+  	  rpy="${mr_rgbd_R * deg_to_rad} ${mr_rgbd_P * deg_to_rad} ${mr_rgbd_Y * deg_to_rad}" />
     <!-- Pose of optical frame wrt to sensor -->
     <origin
@@ -134,5 +140,4 @@
       rpy="${-90 * deg_to_rad} 0 ${-90 * deg_to_rad}"/>
   </xacro:rgbd_camera>
-</xacro:if>
   <!-- RGB -->
 <!--  <xacro:elp_rgb name="rgb_camera" parent="base">-->

File: robot_description/custom/cameras/rgbd_camera.gazebo.xacro (robot description, xacro)
@@ -57,5 +57,5 @@
             <format>R8G8B8</format>
             <width>3840</width> <!-- 320 -->
-            <height>2160</height> <!-- 240 , 2160 stockbot, 2880 to have 4/3 aspect ratio-->
+            <height>2160</height> <!-- 240 , 2160 stockbot (16/9), 2880 to have 4/3 aspect ratio-->
           </image>
           <clip>

Commit message: todo robust rotation

File: robot_description/custom/cameras/cameras.urdf.xacro (robot description, xacro)
@@ -49,5 +49,5 @@
   <xacro:property name="br_rgbd_x" value="0.0"/>
   <xacro:property name="br_rgbd_y" value="${-support_y/2}"/>
-  <xacro:property name="br_rgbd_z" value="${1/3*robot_height - base_height}"/>
+  <xacro:property name="br_rgbd_z" value="${1/3*robot_height - 2*base_height}"/>
   <xacro:property name="br_rgbd_R" value="0.0"/>
   <xacro:property name="br_rgbd_P" value="0.0"/><!-- 10.0-->

Commit message: working alingment, synchronize cameras

File: robot_description/custom/cameras/cameras.urdf.xacro (robot description, xacro)
@@ -28,5 +28,5 @@
   <xacro:property name="ml_rgbd_x" value="0.0"/>
   <xacro:property name="ml_rgbd_y" value="${support_y/2}"/>
-  <xacro:property name="ml_rgbd_z" value="${2/3*robot_height - base_height}"/>
+  <xacro:property name="ml_rgbd_z" value="${2/3*robot_height - 2*base_height}"/>
   <xacro:property name="ml_rgbd_R" value="0.0"/> <!-- rotations are with respect world axis-->
   <xacro:property name="ml_rgbd_P" value="0.0"/><!-- -10.0-->
@@ -35,5 +35,5 @@
   <xacro:property name="mr_rgbd_x" value="0.0"/>
   <xacro:property name="mr_rgbd_y" value="${-support_y/2}"/>
-  <xacro:property name="mr_rgbd_z" value="${2/3*robot_height - base_height}"/>
+  <xacro:property name="mr_rgbd_z" value="${2/3*robot_height - 2*base_height}"/>
   <xacro:property name="mr_rgbd_R" value="0.0"/>
   <xacro:property name="mr_rgbd_P" value="0.0"/><!-- -10.0-->
@@ -42,5 +42,5 @@
   <xacro:property name="bl_rgbd_x" value="0.0"/>
   <xacro:property name="bl_rgbd_y" value="${support_y/2}"/>
-  <xacro:property name="bl_rgbd_z" value="${1/3*robot_height - base_height}"/>
+  <xacro:property name="bl_rgbd_z" value="${base_height + 0.05}"/>
   <xacro:property name="bl_rgbd_R" value="0.0"/>
   <xacro:property name="bl_rgbd_P" value="0.0"/><!-- 10.0-->
@@ -49,5 +49,5 @@
   <xacro:property name="br_rgbd_x" value="0.0"/>
   <xacro:property name="br_rgbd_y" value="${-support_y/2}"/>
-  <xacro:property name="br_rgbd_z" value="${1/3*robot_height - 2*base_height}"/>
+  <xacro:property name="br_rgbd_z" value="${base_height + 0.05}"/>
   <xacro:property name="br_rgbd_R" value="0.0"/>
   <xacro:property name="br_rgbd_P" value="0.0"/><!-- 10.0-->
